Commit message: Use mimic joint

File: ewellix_description/urdf/ewellix_macro.xacro (robot description, xacro)
@@ -157,4 +157,5 @@
       </material>
     </xacro:ewellix_link>
+    <!--
     <joint name="${tf_prefix}upper_joint" type="prismatic">
       <child link="${tf_prefix}upper_link"/>
@@ -170,4 +171,20 @@
       <axis xyz="0 0 1"/>
       <dynamics friction="0.0" damping="0.0"/>
+    </joint>
+     -->
+    <joint name="${tf_prefix}upper_joint" type="prismatic">
+      <child link="${tf_prefix}upper_link"/>
+      <parent link="${tf_prefix}lower_link"/>
+      <origin
+        xyz="0.0 0.0 ${parameters.upper.offset}"
+        rpy="0.0 0.0 0.0"/>
+      <limit
+        effort="${parameters.upper.joint.limit.effort * 1000}"
+        lower="${parameters.upper.joint.limit.lower}"
+        upper="${parameters.upper.joint.limit.upper}"
+        velocity="${parameters.upper.joint.limit.velocity}"/>
+      <axis xyz="0 0 1"/>
+      <dynamics friction="0.0" damping="0.0"/>
+      <mimic joint="${tf_prefix}lower_joint"/>
     </joint>
     <!-- Mount -->
@@ -204,5 +221,4 @@
         <joint name="${tf_prefix}lower_joint">
           <command_interface name="position"/>
-          <!-- <command_interface name="velocity"/> -->
           <state_interface name="position">
             <param name="initial_value">0.0001</param>
@@ -211,7 +227,6 @@
           <state_interface name="effort"/>
         </joint>
-        <joint name="${tf_prefix}upper_joint">
+        <!-- <joint name="${tf_prefix}upper_joint">
           <command_interface name="position"/>
-          <!-- <command_interface name="velocity"/> -->
           <state_interface name="position">
             <param name="initial_value">0.0001</param>
@@ -219,5 +234,5 @@
           <state_interface name="velocity"/>
           <state_interface name="effort"/>
-        </joint>
+        </joint> -->
       </ros2_control>
     </xacro:if>

Commit message: Updated URDF and MoveIt for mimic joint

File: ewellix_description/urdf/ewellix_macro.xacro (robot description, xacro)
@@ -179,4 +179,5 @@
         xyz="0.0 0.0 ${parameters.upper.offset}"
         rpy="0.0 0.0 0.0"/>
+      <axis xyz="0 0 1"/>
       <limit
         effort="${parameters.upper.joint.limit.effort * 1000}"
@@ -184,5 +185,4 @@
         upper="${parameters.upper.joint.limit.upper}"
         velocity="${parameters.upper.joint.limit.velocity}"/>
-      <axis xyz="0 0 1"/>
       <dynamics friction="0.0" damping="0.0"/>
       <mimic joint="${tf_prefix}lower_joint"/>
@@ -227,12 +227,10 @@
           <state_interface name="effort"/>
         </joint>
-        <!-- <joint name="${tf_prefix}upper_joint">
-          <command_interface name="position"/>
-          <state_interface name="position">
-            <param name="initial_value">0.0001</param>
-          </state_interface>
-          <state_interface name="velocity"/>
-          <state_interface name="effort"/>
-        </joint> -->
+        <xacro:if value="${sim_ignition or use_fake_hardware}">
+          <joint name="${tf_prefix}upper_joint">
+            <param name="mimic">${tf_prefix}lower_joint</param>
+            <param name="multiplier">1</param>
+          </joint>
+        </xacro:if>
       </ros2_control>
     </xacro:if>

Commit message: Add friction and initialize lift extended

File: ewellix_description/urdf/ewellix_macro.xacro (robot description, xacro)
@@ -139,10 +139,10 @@
         rpy="0.0 0.0 0.0"/>
       <limit
-        effort="${parameters.lower.joint.limit.effort * 1000}"
+        effort="${parameters.lower.joint.limit.effort}"
         lower="${parameters.lower.joint.limit.lower}"
         upper="${parameters.lower.joint.limit.upper}"
         velocity="${parameters.lower.joint.limit.velocity}"/>
       <axis xyz="0 0 1"/>
-      <dynamics friction="0.0" damping="0.0"/>
+      <dynamics friction="0.01" damping="0.01"/>
     </joint>
     <!-- Upper Tower -->
@@ -157,20 +157,4 @@
       </material>
     </xacro:ewellix_link>
-    <!--
-    <joint name="${tf_prefix}upper_joint" type="prismatic">
-      <child link="${tf_prefix}upper_link"/>
-      <parent link="${tf_prefix}lower_link"/>
-      <origin
-        xyz="0.0 0.0 ${parameters.upper.offset}"
-        rpy="0.0 0.0 0.0"/>
-      <limit
-        effort="${parameters.upper.joint.limit.effort * 1000}"
-        lower="${parameters.upper.joint.limit.lower}"
-        upper="${parameters.upper.joint.limit.upper}"
-        velocity="${parameters.upper.joint.limit.velocity}"/>
-      <axis xyz="0 0 1"/>
-      <dynamics friction="0.0" damping="0.0"/>
-    </joint>
-     -->
     <joint name="${tf_prefix}upper_joint" type="prismatic">
       <child link="${tf_prefix}upper_link"/>
@@ -181,9 +165,9 @@
       <axis xyz="0 0 1"/>
       <limit
-        effort="${parameters.upper.joint.limit.effort * 1000}"
+        effort="${parameters.upper.joint.limit.effort}"
         lower="${parameters.upper.joint.limit.lower}"
         upper="${parameters.upper.joint.limit.upper}"
         velocity="${parameters.upper.joint.limit.velocity}"/>
-      <dynamics friction="0.0" damping="0.0"/>
+      <dynamics friction="0.01" damping="0.01"/>
       <mimic joint="${tf_prefix}lower_joint"/>
     </joint>
@@ -222,5 +206,5 @@
           <command_interface name="position"/>
           <state_interface name="position">
-            <param name="initial_value">0.0001</param>
+            <param name="initial_value">${parameters.lower.joint.limit.upper}</param>
           </state_interface>
           <state_interface name="velocity"/>

Commit message: Add mount plate mesh

File: ewellix_description/urdf/ewellix_macro.xacro (robot description, xacro)
@@ -173,12 +173,43 @@
     </joint>
     <!-- Mount -->
-    <link name="${tf_prefix}mount"/>
-    <joint name="${tf_prefix}mount_joint" type="fixed">
-      <child link="${tf_prefix}mount"/>
-      <parent link="${tf_prefix}upper_link"/>
-      <origin
-        xyz="0.0 0.0 ${fabs(parameters.upper.max.z - parameters.upper.min.z)}"
-        rpy="0.0 0.0 0.0"/>
-    </joint>
+    <xacro:if value="${parameters.get('mount')}">
+      <!-- Mount: Arm Mounting Plate -->
+      <xacro:ewellix_link
+        name="${tf_prefix}mount_link"
+        mesh="package://ewellix_description/meshes/${parameters.mount.mesh}"
+        maximum="${parameters.mount.max}"
+        minimum="${parameters.mount.min}"
+        mass="${parameters.mount.mass}">
+        <material name="${parameters.mount.material.name}">
+        <color rgba="${parameters.mount.material.color}"/>
+        </material>
+      </xacro:ewellix_link>
+      <joint name="${tf_prefix}_mount_link_joint" type="fixed">
+        <child link="${tf_prefix}mount_link"/>
+        <parent link="${tf_prefix}upper_link"/>
+        <origin
+          xyz="0.0 0.0 ${fabs(parameters.upper.max.z - parameters.upper.min.z) + parameters.mount.offset}"
+          rpy="0.0 0.0 0.0"/>
+      </joint>
+      <link name="${tf_prefix}mount"/>
+      <joint name="${tf_prefix}mount_joint" type="fixed">
+        <child link="${tf_prefix}mount"/>
+        <parent link="${tf_prefix}mount_link"/>
+        <origin
+          xyz="0.0 0.0 ${fabs(parameters.mount.max.z - parameters.mount.min.z)}"
+          rpy="0.0 0.0 0.0"/>
+      </joint>
+    </xacro:if>
+    <xacro:unless value="${parameters.get('mount')}">
+      <!-- Mount: Virtual Link -->
+      <link name="${tf_prefix}mount"/>
+      <joint name="${tf_prefix}mount_joint" type="fixed">
+        <child link="${tf_prefix}mount"/>
+        <parent link="${tf_prefix}upper_link"/>
+        <origin
+          xyz="0.0 0.0 ${fabs(parameters.upper.max.z - parameters.upper.min.z)}"
+          rpy="0.0 0.0 0.0"/>
+      </joint>
+    </xacro:unless>
     <!-- ROS 2 Controls -->
     <xacro:if value="${generate_ros2_control_tag}">
